File: AuxPCB/AuxRelays.kicad_sch (KiCad schematic)
At the start: 0 parts

Commit message: Started schematic
Parts:
- added D1, D10, D11, D12, D13, D14, D15, D16, D17, D18, D19, D2, D20, D3, D4, D5, D6, D7, D8, D9: SMA, Diode_SMD:D_SMA, symbol Device:D_Filled
- added J1, J2, J3: Conn_01x10, TerminalBlock_Phoenix:TerminalBlock_Phoenix_PT-1,5-10-3.5-H_1x10_P3.50mm_Horizontal, symbol Connector_Generic:Conn_01x10
- added LED1, LED2: LED, LED_SMD:LED_1206_3216Metric_Pad1.42x1.75mm_HandSolder, symbol Device:LED_Filled
- added Q1, Q2: IRF7343PBF, Package_SO:SOIC-8_3.9x4.9mm_P1.27mm, symbol Transistor_FET:IRF7343PBF
- added R1, R10, R2, R3, R4, R5, R6, R7, R8, R9: 10K, Resistor_SMD:R_0805_2012Metric_Pad1.20x1.40mm_HandSolder, symbol Device:R_Small
Connections:
- new net: Q2.5 (D), Q2.6 (D)
- new net: Q2.7 (D), Q2.8 (D)
- new net: Q1.5 (D), Q1.6 (D)
- new net: Q1.7 (D), Q1.8 (D)
Other:
- note added: "OCC24 T-In T-In Grn Red Wht Bid R Bid G FBR BID"
- note added: "OCC24* T-In T-In Grn Red Wht Bid R Bid G FBR BID"
- note added: "TRK TRK GND GND InUse24 InUse24* BlkInUse"

Commit message: Done and OSHPARKed
Parts:
- added D14, D3: SMA, Diode_SMD:D_SMA, symbol Device:D_Filled
- added RLY1, RLY2: MY4PDT, MY4PDT:MY4PDT, symbol MY4PDT:MY4PDT
- renumbered D9 to D1, D7 to D11, D19 to D12, D15 to D13, D14 to D15, D13 to D16, D12 to D17, D11 to D18, D16 to D19, D5 to D2, D18 to D20, D20 to D21, D17 to D22, D3 to D5, D2 to D6, D1 to D7, D6 to D8, D8 to D9
Connections:
- net at LED2.1 (K): now also D13.2 (A), D18.2 (A), J2.2 (Pin_2), Q2.1 (S), R8.1, RLY2.13
- net at LED2.2 (A): now also R6.2
- net GND: now reaches Q2.3 (1)
- net GND: now also J3.7 (Pin_7), J3.8 (Pin_8), Q1.3 (1), R10.1, R5.1
- net at Q2.4 (G): now also R10.2, R9.1
- net at Q2.5 (D), Q2.6 (D): now also D12.1 (K), D21.1 (K)
- net at D13.1 (K): now also D19.1 (K), D20.1 (K), R6.1, RLY2.14
- net at Q2.2 (G): now also D12.2 (A), R7.1, R8.2
- net at Q2.7 (D), Q2.8 (D): now also D14.1 (K)
- net at R2.1: now also D1.2 (A), Q1.2 (G), R3.2
- net at R2.2: now also J3.4 (Pin_4), R7.2
- net at LED1.1 (K): now also D2.2 (A), D7.2 (A), J1.2 (Pin_2), Q1.1 (S), R3.1, RLY1.13
- net at LED1.2 (A): now also R1.2
- net at Q1.4 (G): now also R4.1, R5.2
- net at Q1.5 (D), Q1.6 (D): now also D1.1 (K), D10.1 (K)
- net at D19.2 (A): now also D22.2 (A), R9.2, RLY2.8
- net at D4.1 (K): now also J1.7 (Pin_7)
- net at D4.2 (A): now also RLY1.6
- net at D18.1 (K): now also J2.1 (Pin_1)
- net at D8.1 (K): now also D2.1 (K), D9.1 (K), R1.1, RLY1.14
- net at D8.2 (A): now also D11.2 (A), R4.2, RLY1.8
- net at Q1.7 (D), Q1.8 (D): now also D3.1 (K)
- net at D7.1 (K): now also J1.1 (Pin_1)
- net at J3.1 (Pin_1): now also RLY1.12
- net at J3.10 (Pin_10): now also J3.9 (Pin_9), RLY1.9, RLY2.9
- net at J3.2 (Pin_2): now also D11.1 (K), D22.1 (K)
- net at J3.3 (Pin_3): now also D20.2 (A), D9.2 (A)
- net at J3.5 (Pin_5): now also RLY2.4
- net at D21.2 (A): now also J2.3 (Pin_3)
- net at D15.1 (K): now also J2.7 (Pin_7)
- net at D15.2 (A): now also RLY2.6
- net at D16.1 (K): now also J2.6 (Pin_6)
- net at D16.2 (A): now also RLY2.3
- net at J1.10 (Pin_10): now also RLY1.10, RLY2.10
- net at J1.3 (Pin_3): now also D10.2 (A)
- net at J1.4 (Pin_4): now also D3.2 (A)
- net at J1.5 (Pin_5): now also D6.1 (K)
- net at J1.6 (Pin_6): now also D5.1 (K)
- net at J1.8 (Pin_8): now also J1.9 (Pin_9), RLY1.5
- net at J2.10 (Pin_10): now also RLY1.11, RLY2.11
- net at J2.4 (Pin_4): now also D14.2 (A)
- net at J2.5 (Pin_5): now also D17.1 (K)
- net at J2.8 (Pin_8): now also J2.9 (Pin_9), RLY2.5
- net at D5.2 (A): now also RLY1.3
- net at D17.2 (A): now also RLY2.7
- net at D6.2 (A): now also RLY1.7
- new net: RLY1.4, RLY2.12
- no-connect marks 0 -> 5
Other:
- note added: "ENA connects to NXTCAB of previous board or +24VDC if used stand-alone. Main Secondary (This PCB) Occ24* >> Occ24* J1-10 Occ24 >> Occ24 J2-10 NXTCAB >> Enable +24 J3-1 BlkInUse << BlkInUse J3-2 InUse24 >> InUse24 J3-4 InUse24* >> InUse24* J3-3"
- note added: "TRK TRK GND GND NXTCAB InUse24 InUse24* BlkInUse ENA"
- note removed: "TRK TRK GND GND InUse24 InUse24* BlkInUse"
- moved on the sheet: D1, D10, D11, D12, D13, D15, D16, D17, D18, D19, D2, D20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
